Commit message: added camera urdf

File: urdf/lidar.xacro (robot description, xacro)
@@ -23,7 +23,8 @@
     </link>
     <gazebo reference="laser_frame">
+        <material>Gazebo/Red</material>
         <sensor name="laser" type="gpu_lidar">
             <pose> 0 0 0 0 0 0 </pose>
-            <visualize>true</visualize>
+            <visualize>false</visualize>
             <update_rate>10</update_rate>
             <lidar>

File: urdf/robot.urdf.xacro (robot description, xacro)
@@ -4,3 +4,4 @@
     <xacro:include filename="ros2_control.xacro"/>
     <xacro:include filename="lidar.xacro"/>
+    <xacro:include filename="camera.xacro"/>
 </robot>
