Commit message: added ros2 control plugin

File: urdf/robot_core.xacro (robot description, xacro)
@@ -120,4 +120,6 @@
     <gazebo reference="caster_wheel">
         <material>Gazebo/Black</material>
+        <mu1 value="0.001"/>
+        <mu2 value="0.001"/>
     </gazebo>
 </robot>

File: urdf/ros2_control.xacro (robot description, xacro)
@@ -1,8 +1,28 @@
 <?xml version="1.0"?>
 <robot xmlns:xacro="http://ros.org/wiki/xacro">
-    <ros2_control name="GazeboSystem" type="system">
+    <ros2_control name="GazeboSimSystem" type="system">
         <hardware>
-            <plugin></plugin>
+            <plugin>gz_ros2_control/GazeboSimSystem</plugin>
         </hardware>
+        <joint name="left_wheel_joint">
+            <command_interface name="velocity"></command_interface>
+            <state_interface name="velocity"></state_interface>
+            <state_interface name="position"/>
+        </joint>
+        <joint name="right_wheel_joint">
+            <command_interface name="velocity"></command_interface>
+            <state_interface name="velocity"></state_interface>
+            <state_interface name="position"/>
+        </joint>
     </ros2_control>
+    <gazebo>
+        <plugin filename="gz_ros2_control-system" name="gz_ros2_control::GazeboSimROS2ControlPlugin">
+            <ros>
+                <namespace>/</namespace>
+            </ros>
+            <robot_param>robot_description</robot_param>
+            <robot_param_node>robot_state_publisher</robot_param_node>
+            <parameters>$(find dd_bot)/config/controllers.yaml</parameters>
+        </plugin>
+    </gazebo>
 </robot>

Commit message: added slam toolbox package and obstacle world

File: urdf/robot_core.xacro (robot description, xacro)
@@ -19,4 +19,11 @@
     <!-- Base link -->
     <link name="base_link">
+    </link>
+    <joint name="base_footprint_joint" type="fixed">
+        <parent link="base_link"/>
+        <child link="base_footprint"/>
+        <origin xyz="0 0 0" rpy="0 0 0"/>
+    </joint>
+    <link name="base_footprint">
     </link>
     <!-- Chassis link -->
